Commit message: control

File: g_vehicle/car_v3.urdf (robot description, URDF)
Before this commit: robot car, 14 links, 13 joints
Links:
- link H_left: geometry collision box size=${r_circle*h_h} ${r_circle*h_w/4.25} ${t}; visual box size=${r_circle*h_h} ${r_circle*h_w/4.25} ${t}
- link H_middle: geometry collision box size=${r_circle*h_h*0.8/3.4} ${r_circle*h_w*2.0/3.4} ${t}; visual box size=${r_circle*h_h*0.8/3.4} ${r_circle*h_w*2.0/3.4} ${t}
- link H_right: geometry collision box size=${r_circle*h_h} ${r_circle*h_w/4.25} ${t}; visual box size=${r_circle*h_h} ${r_circle*h_w/4.25} ${t}
- link back_left_wheel_link: mass 0.01 -> None; geometry 
- link back_right_wheel_link: mass 0.01 -> None; geometry 
- link bar_link: mass 0.01 -> ${0.01*k_car**3}; geometry collision cylinder length=${0.2*k_car} radius=${0.01*k_car}; visual cylinder length=${0.175*k_car} radius=${0.01*k_car}
- link base_link: mass 0.2 -> ${0.2*k_car**3}
- link front_left_wheel_link: mass 0.01 -> None; geometry 
- link front_right_wheel_link: mass 0.01 -> None; geometry 
- link heliport_base: mass 0.00040000000000000013 -> ${0.05*a_base**3}; geometry collision box size=${a_base} ${a_base} ${0.025*a_base}; visual box size=${a_base} ${a_base} ${0.025*a_base}
- link heliport_circle: geometry collision cylinder length=${t} radius=${r_circle}; visual cylinder length=${t} radius=${r_circle}
- link holder: mass 0.01 -> ${0.01*k_car**3}; geometry collision cylinder length=${0.05*k_car} radius=${0.005*k_car}; visual cylinder length=${0.05*k_car} radius=${0.005*k_car}
- link main_body: mass 0.2 -> ${0.2*k_car**3}; geometry collision box size=${0.3*k_car} ${0.15*k_car} ${0.1*k_car}; visual box size=${0.3*k_car} ${0.15*k_car} ${0.1*k_car}
- link rear_bar_link: mass 0.01 -> ${0.01*k_car**3}; geometry collision cylinder length=${0.2*k_car} radius=${0.01*k_car}; visual cylinder length=${0.175*k_car} radius=${0.01*k_car}
Joints:
- joint H_left_to_circle: origin xyz=0 0.020588235294117647 0.001 rpy=0 0 0 -> xyz=0 ${r_circle*h_w*1.4/3.4} ${t} rpy=0 0 0
- joint H_middle_to_circle: origin xyz=0 0 0.001 rpy=0 0 0 -> xyz=0 0 ${t} rpy=0 0 0
- joint H_right_to_circle: origin xyz=0 -0.020588235294117647 0.001 rpy=0 0 0 -> xyz=0 -${r_circle*h_w*1.4/3.4} ${t} rpy=0 0 0
- joint back_left_wheel_joint: origin xyz=0.0 0.0 0.1 rpy=1.5707963267948966 0 0 -> xyz=0.0 0.0 ${0.1*k_car} rpy=${pi/2} 0 0
- joint back_right_wheel_joint: origin xyz=0.0 0.0 -0.1 rpy=1.5707963267948966 0 0 -> xyz=0.0 0.0 ${-0.1*k_car} rpy=${pi/2} 0 0
- joint bar_joint: origin xyz=0.16 0.0 -0.1 rpy=-1.5707963267948966 0 0 -> xyz=${0.16*k_car} 0.0 ${-0.1*k_car} rpy=${-pi/2} 0 0
- joint base_to_holder: origin xyz=0 0 0.075 rpy=0 0 0 -> xyz=0 0 ${0.075*k_car} rpy=0 0 0
- joint dummy: origin xyz=0 0 0.16 rpy=0 0 0 -> xyz=0 0 ${0.16*k_car} rpy=0 0 0
- joint front_left_wheel_joint: origin xyz=0.0 0.0 -0.1 rpy=1.5707963267948966 0 0 -> xyz=0.0 0.0 ${-0.1*k_car} rpy=${pi/2} 0 0
- joint front_right_wheel_joint: origin xyz=0.0 0.0 0.1 rpy=1.5707963267948966 0 0 -> xyz=0.0 0.0 ${0.1*k_car} rpy=${pi/2} 0 0
- joint heliport_base_to_circle: origin xyz=0 0 0.0030000000000000005 rpy=0 0 0 -> xyz=0 0 ${0.0125*a_base+t/2} rpy=0 0 0
- joint holder_to_heliport: origin xyz=0 0 0.027500000000000004 rpy=0 0 0 -> xyz=0 0 ${0.025*k_car+0.0125*a_base} rpy=0 0 0
- joint rear_bar_joint: origin xyz=-0.16 0.0 -0.1 rpy=-1.5707963267948966 0 0 -> xyz=${-0.16*k_car} 0.0 ${-0.1*k_car} rpy=${-pi/2} 0 0
