Commit message: working crazy fly

File: g_vehicle/parsed.urdf (robot description, URDF)
Before this commit: robot car, 14 links, 13 joints
Links:
- link H_left: geometry collision box size=0.35000000000000003 0.0823529411764706 0.001; visual box size=0.35000000000000003 0.0823529411764706 0.001
- link H_middle: geometry collision box size=0.0823529411764706 0.2058823529411765 0.001; visual box size=0.0823529411764706 0.2058823529411765 0.001
- link H_right: geometry collision box size=0.35000000000000003 0.0823529411764706 0.001; visual box size=0.35000000000000003 0.0823529411764706 0.001
- link heliport_base: mass 0.00040000000000000013 -> 0.05; geometry collision box size=1.0 1.0 0.025; visual box size=1.0 1.0 0.025
- link heliport_circle: geometry collision cylinder length=0.001 radius=0.35000000000000003; visual cylinder length=0.001 radius=0.35000000000000003
Joints:
- joint H_left_to_circle: origin xyz=0 0.020588235294117647 0.001 rpy=0 0 0 -> xyz=0 0.14411764705882352 0.001 rpy=0 0 0
- joint H_right_to_circle: origin xyz=0 -0.020588235294117647 0.001 rpy=0 0 0 -> xyz=0 -0.14411764705882352 0.001 rpy=0 0 0
- joint heliport_base_to_circle: origin xyz=0 0 0.0030000000000000005 rpy=0 0 0 -> xyz=0 0 0.013000000000000001 rpy=0 0 0
- joint holder_to_heliport: origin xyz=0 0 0.027500000000000004 rpy=0 0 0 -> xyz=0 0 0.037500000000000006 rpy=0 0 0

Commit message: changes

File: g_vehicle/parsed.urdf (robot description, URDF)
Before this commit: robot car, 14 links, 13 joints
Links:
- link H_left: geometry collision box size=0.35000000000000003 0.0823529411764706 0.001; visual box size=0.35000000000000003 0.0823529411764706 0.001
- link H_middle: geometry collision box size=0.0823529411764706 0.2058823529411765 0.001; visual box size=0.0823529411764706 0.2058823529411765 0.001
- link H_right: geometry collision box size=0.35000000000000003 0.0823529411764706 0.001; visual box size=0.35000000000000003 0.0823529411764706 0.001
- link heliport_base: mass 0.00040000000000000013 -> 0.05; geometry collision box size=1.0 1.0 0.025; visual box size=1.0 1.0 0.025
- link heliport_circle: geometry collision cylinder length=0.001 radius=0.35000000000000003; visual cylinder length=0.001 radius=0.35000000000000003
Joints:
- joint H_left_to_circle: origin xyz=0 0.020588235294117647 0.001 rpy=0 0 0 -> xyz=0 0.14411764705882352 0.001 rpy=0 0 0
- joint H_right_to_circle: origin xyz=0 -0.020588235294117647 0.001 rpy=0 0 0 -> xyz=0 -0.14411764705882352 0.001 rpy=0 0 0
- joint heliport_base_to_circle: origin xyz=0 0 0.0030000000000000005 rpy=0 0 0 -> xyz=0 0 0.013000000000000001 rpy=0 0 0
- joint holder_to_heliport: origin xyz=0 0 0.027500000000000004 rpy=0 0 0 -> xyz=0 0 0.037500000000000006 rpy=0 0 0; type spherical -> fixed
